Commit message: Fixed some issues with indigo migration

File: calf_description/urdf/base.urdf.xacro (robot description, xacro)
@@ -115,7 +115,8 @@
       <transmission name="${robot_ns}/left_drive_trans">
         <type>transmission_interface/SimpleTransmission</type>
-        <joint name="${robot_ns}/left_drive_joint"/>
+        <joint name="${robot_ns}/left_drive_joint">
+          <hardwareInterface>EffortJointInterface</hardwareInterface>
+	</joint>
         <actuator name="${robot_ns}/left_drive_actuator">
-          <hardwareInterface>EffortJointInterface</hardwareInterface>
           <mechanicalReduction>1</mechanicalReduction>
         </actuator>
@@ -123,7 +124,8 @@
       <transmission name="${robot_ns}/right_drive_trans">
         <type>transmission_interface/SimpleTransmission</type>
-        <joint name="${robot_ns}/right_drive_joint"/>
+        <joint name="${robot_ns}/right_drive_joint">
+          <hardwareInterface>EffortJointInterface</hardwareInterface>
+	</joint>
         <actuator name="${robot_ns}/right_drive_actuator">
-          <hardwareInterface>EffortJointInterface</hardwareInterface>
           <mechanicalReduction>1</mechanicalReduction>
         </actuator>

File: calf_description/urdf/pod.urdf.xacro (robot description, xacro)
@@ -38,7 +38,8 @@
 		<transmission name="${robot_ns}/${fb}_${lr}_pod_joint_trans">
 			<type>transmission_interface/SimpleTransmission</type>
-			<joint name="${robot_ns}/${fb}_${lr}_pod_joint"/>
+			<joint name="${robot_ns}/${fb}_${lr}_pod_joint">
+				<hardwareInterface>EffortJointInterface</hardwareInterface>
+			</joint>
 			<actuator name="${robot_ns}/${fb}_${lr}_pod_joint_actuator">
-				<hardwareInterface>EffortJointInterface</hardwareInterface>
 				<mechanicalReduction>1</mechanicalReduction>
 			</actuator>
