Commit message: First pass at a gazebo WALRUS gazebo plugin

File: walrus_description/robots/walrus.urdf.xacro (robot description, xacro)
@@ -6,9 +6,9 @@
   <property name="robot_ns" value="walrus" />
   <xacro:walrus robot_ns="${robot_ns}"/>
-  <!--<gazebo>
+  <gazebo>
     <plugin name="gazebo_ros_control" filename="libgazebo_ros_control.so">
       <robotNamespace>/walrus</robotNamespace>
       <robotSimType>walrus_gazebo/WalrusHWSim</robotSimType>
     </plugin>
-  </gazebo>-->
+  </gazebo>
 </robot>

File: walrus_description/urdf/center_tread.urdf.xacro (robot description, xacro)
@@ -93,5 +93,5 @@
 			</collision>
 		</link>
-		<joint name="${robot_ns}/${lr}_center_tread_back_cylinder_joint" type="continuous">
+		<joint name="${robot_ns}/${lr}_drive_idler_joint" type="continuous">
 			<parent link="${robot_ns}/${lr}_center_tread"/>
 			<child link="${robot_ns}/${lr}_center_tread_back_cylinder"/>

File: walrus_description/urdf/pod.urdf.xacro (robot description, xacro)
@@ -45,5 +45,5 @@
 			</actuator>
 		</transmission>
-		<link name="${robot_ns}/${fb}_${lr}_pod_joint_cylinder">
+		<link name="${robot_ns}/${fb}_${lr}_pod_drive_cylinder">
 			<inertial>
 				<mass value="${tread_cylinder_mass}" />
@@ -74,12 +74,12 @@
 			</collision>
 		</link>
-		<joint name="${robot_ns}/${fb}_${lr}_pod_joint_cylinder_joint" type="continuous">
+		<joint name="${robot_ns}/${fb}_${lr}_pod_drive_joint" type="continuous">
 			<parent link="${robot_ns}/${fb}_${lr}_pod"/>
-			<child link="${robot_ns}/${fb}_${lr}_pod_joint_cylinder"/>
+			<child link="${robot_ns}/${fb}_${lr}_pod_drive_cylinder"/>
 			<origin xyz="0 0 0" rpy="${M_PI/2} 0 0" />
 			<axis xyz="0 0 1" rpy="0 0 0" />
 			<mimic joint="${robot_ns}/${lr}_drive_joint" multiplier="1.0" offset="0.0" />
 		</joint>
-		<link name="${robot_ns}/${fb}_${lr}_pod_extended_cylinder">
+		<link name="${robot_ns}/${fb}_${lr}_pod_drive_idler_cylinder">
 			<inertial>
 				<mass value="${tread_cylinder_mass}" />
@@ -110,7 +110,7 @@
 			</collision>
 		</link>
-		<joint name="${robot_ns}/${fb}_${lr}_pod_extended_cylinder_joint" type="continuous">
+		<joint name="${robot_ns}/${fb}_${lr}_pod_drive_idler_joint" type="continuous">
 			<parent link="${robot_ns}/${fb}_${lr}_pod"/>
-			<child link="${robot_ns}/${fb}_${lr}_pod_extended_cylinder"/>
+			<child link="${robot_ns}/${fb}_${lr}_pod_drive_idler_cylinder"/>
 			<origin xyz="${pod_inner_length} 0 0" rpy="${M_PI/2} 0 0" />
 			<axis xyz="0 0 1" rpy="0 0 0" />

Commit message: Cleaned up tf namespacing

File: walrus_description/robots/walrus.urdf.xacro (robot description, xacro)
@@ -1,11 +1,12 @@
 <?xml version="1.0"?>
-<robot name="walrus" xmlns:xacro="http://ros.org/wiki/xacro">
+<robot name="$(arg robot_name)" xmlns:xacro="http://ros.org/wiki/xacro">
   <!-- Included URDF/XACRO Files -->
   <xacro:include filename="$(find walrus_description)/urdf/base.urdf.xacro" />
-  <property name="robot_ns" value="walrus" />
-  <xacro:walrus robot_ns="${robot_ns}"/>
+  <property name="tf_prefix" value="$(arg tf_prefix)" />
+  <property name="robot_ns" value="$(arg robot_ns)" />
+  <xacro:walrus tf_prefix="${tf_prefix}"/>
   <gazebo>
     <plugin name="gazebo_ros_control" filename="libgazebo_ros_control.so">
-      <robotNamespace>/walrus</robotNamespace>
+      <robotNamespace>${robot_ns}</robotNamespace>
       <robotSimType>walrus_gazebo/WalrusHWSim</robotSimType>
     </plugin>

File: walrus_description/urdf/base.urdf.xacro (robot description, xacro)
@@ -62,7 +62,7 @@
     <xacro:include filename="$(find walrus_description)/urdf/pod.urdf.xacro" />
     <xacro:include filename="$(find walrus_description)/urdf/center_tread.urdf.xacro" />
-    <xacro:macro name="walrus" params="robot_ns">
+    <xacro:macro name="walrus" params="tf_prefix">
       <!-- BASE-FOOTPRINT -->
-      <link name="${robot_ns}/base_footprint">
+      <link name="${tf_prefix}base_footprint">
 	<visual>
 	  <origin xyz="0 0 0" rpy="0 0 0" />
@@ -72,15 +72,15 @@
 	</visual>
       </link>
-      <gazebo reference="${robot_ns}/base_footprint">
+      <gazebo reference="${tf_prefix}base_footprint">
 	<turnGravityOff>false</turnGravityOff>
       </gazebo>
-      <joint name="${robot_ns}/base_link_joint" type="fixed">
+      <joint name="${tf_prefix}base_link_joint" type="fixed">
 	<origin xyz="0 0 ${tread_radius + base_z_to_pod_origin}" rpy="0 0 0" />
-	<parent link="${robot_ns}/base_footprint"/>
-	<child link="${robot_ns}/base_link" />
+	<parent link="${tf_prefix}base_footprint"/>
+	<child link="${tf_prefix}base_link" />
       </joint>
       <!-- BASE-LINK -->
       <!--Actual body/chassis of the robot-->
-      <link name="${robot_ns}/base_link">
+      <link name="${tf_prefix}base_link">
 	<inertial>
 	  <mass value="${base_mass}" />
@@ -103,29 +103,29 @@
 	</collision>
       </link>
-      <gazebo reference="${robot_ns}/base_link">
+      <gazebo reference="${tf_prefix}base_link">
 	<material>Gazebo/Green</material>
 	<turnGravityOff>false</turnGravityOff>
       </gazebo>
-      <walrus_pod fb="back" lr="left" parent="${robot_ns}/base_link" translateX="-1" translateY="1" flipY="-1" robot_ns="${robot_ns}"/>
-      <walrus_pod fb="back" lr="right" parent="${robot_ns}/base_link" translateX="-1" translateY="-1" flipY="-1" robot_ns="${robot_ns}"/>
-      <walrus_pod fb="front" lr="left" parent="${robot_ns}/base_link" translateX="1" translateY="1" flipY="-1" robot_ns="${robot_ns}"/>
-      <walrus_pod fb="front" lr="right" parent="${robot_ns}/base_link" translateX="1" translateY="-1" flipY="-1" robot_ns="${robot_ns}"/>
-      <walrus_center_tread lr="left" parent="${robot_ns}/base_link" translateY="1" flipY="-1" robot_ns="${robot_ns}"/>
-      <walrus_center_tread lr="right" parent="${robot_ns}/base_link" translateY="-1" flipY="-1" robot_ns="${robot_ns}"/>
-      <transmission name="${robot_ns}/left_drive_trans">
+      <walrus_pod fb="back" lr="left" parent="${tf_prefix}base_link" translateX="-1" translateY="1" flipY="-1" tf_prefix="${tf_prefix}"/>
+      <walrus_pod fb="back" lr="right" parent="${tf_prefix}base_link" translateX="-1" translateY="-1" flipY="-1" tf_prefix="${tf_prefix}"/>
+      <walrus_pod fb="front" lr="left" parent="${tf_prefix}base_link" translateX="1" translateY="1" flipY="-1" tf_prefix="${tf_prefix}"/>
+      <walrus_pod fb="front" lr="right" parent="${tf_prefix}base_link" translateX="1" translateY="-1" flipY="-1" tf_prefix="${tf_prefix}"/>
+      <walrus_center_tread lr="left" parent="${tf_prefix}base_link" translateY="1" flipY="-1" tf_prefix="${tf_prefix}"/>
+      <walrus_center_tread lr="right" parent="${tf_prefix}base_link" translateY="-1" flipY="-1" tf_prefix="${tf_prefix}"/>
+      <transmission name="${tf_prefix}left_drive_trans">
         <type>transmission_interface/SimpleTransmission</type>
-        <joint name="${robot_ns}/left_drive_joint">
+        <joint name="${tf_prefix}left_drive_joint">
           <hardwareInterface>hardware_interface/EffortJointInterface</hardwareInterface>
 	</joint>
-        <actuator name="${robot_ns}/left_drive_actuator">
+        <actuator name="${tf_prefix}left_drive_actuator">
           <mechanicalReduction>1</mechanicalReduction>
         </actuator>
       </transmission>
-      <transmission name="${robot_ns}/right_drive_trans">
+      <transmission name="${tf_prefix}right_drive_trans">
         <type>transmission_interface/SimpleTransmission</type>
-        <joint name="${robot_ns}/right_drive_joint">
+        <joint name="${tf_prefix}right_drive_joint">
           <hardwareInterface>hardware_interface/EffortJointInterface</hardwareInterface>
 	</joint>
-        <actuator name="${robot_ns}/right_drive_actuator">
+        <actuator name="${tf_prefix}right_drive_actuator">
           <mechanicalReduction>1</mechanicalReduction>
         </actuator>

File: walrus_description/urdf/center_tread.urdf.xacro (robot description, xacro)
@@ -1,6 +1,6 @@
 <?xml version="1.0"?>
 <robot xmlns:xacro="http://ros.org/wiki/xacro" name="walrus_center_tread">
-	<xacro:macro name="walrus_center_tread" params="lr parent translateY flipY robot_ns"> <!--lr: left, right -->
-		<link name="${robot_ns}/${lr}_center_tread">
+	<xacro:macro name="walrus_center_tread" params="lr parent translateY flipY tf_prefix"> <!--lr: left, right -->
+		<link name="${tf_prefix}${lr}_center_tread">
 			<inertial>
 				<mass value="${center_tread_mass}" />
@@ -24,10 +24,10 @@
 			</collision>
 		</link>
-		<joint name="${robot_ns}/${lr}_center_tread_joint" type="fixed">
+		<joint name="${tf_prefix}${lr}_center_tread_joint" type="fixed">
 			<parent link="${parent}"/>
-			<child link="${robot_ns}/${lr}_center_tread"/>
+			<child link="${tf_prefix}${lr}_center_tread"/>
 			<origin xyz="0 ${translateY * (base_y_size/2+tread_width/2)} ${-base_z_to_pod_origin}" rpy="0 0 0" />
 		</joint>
-		<link name="${robot_ns}/${lr}_center_tread_front_cylinder">
+		<link name="${tf_prefix}${lr}_center_tread_front_cylinder">
 			<inertial>
 				<mass value="${tread_cylinder_mass}" />
@@ -58,11 +58,11 @@
 			</collision>
 		</link>
-		<joint name="${robot_ns}/${lr}_drive_joint" type="continuous">
-			<parent link="${robot_ns}/${lr}_center_tread"/>
-			<child link="${robot_ns}/${lr}_center_tread_front_cylinder"/>
+		<joint name="${tf_prefix}${lr}_drive_joint" type="continuous">
+			<parent link="${tf_prefix}${lr}_center_tread"/>
+			<child link="${tf_prefix}${lr}_center_tread_front_cylinder"/>
 			<origin xyz="${center_tread_inner_length/2} 0 0" rpy="${M_PI/2} 0 0" />
 			<axis xyz="0 0 1" rpy="0 0 0" />
 		</joint>
-		<link name="${robot_ns}/${lr}_center_tread_back_cylinder">
+		<link name="${tf_prefix}${lr}_center_tread_back_cylinder">
 			<inertial>
 				<mass value="${tread_cylinder_mass}" />
@@ -93,10 +93,10 @@
 			</collision>
 		</link>
-		<joint name="${robot_ns}/${lr}_drive_idler_joint" type="continuous">
-			<parent link="${robot_ns}/${lr}_center_tread"/>
-			<child link="${robot_ns}/${lr}_center_tread_back_cylinder"/>
+		<joint name="${tf_prefix}${lr}_drive_idler_joint" type="continuous">
+			<parent link="${tf_prefix}${lr}_center_tread"/>
+			<child link="${tf_prefix}${lr}_center_tread_back_cylinder"/>
 			<origin xyz="${-center_tread_inner_length/2} 0 0" rpy="${M_PI/2} 0 0" />
 			<axis xyz="0 0 1" rpy="0 0 0" />
-			<mimic joint="${robot_ns}/${lr}_drive_joint" multiplier="1.0" offset="0.0" />
+			<mimic joint="${tf_prefix}${lr}_drive_joint" multiplier="1.0" offset="0.0" />
 		</joint>
   	</xacro:macro>

File: walrus_description/urdf/pod.urdf.xacro (robot description, xacro)
@@ -1,6 +1,6 @@
 <?xml version="1.0" encoding="utf-8"?>
 <robot xmlns:xacro="http://ros.org/wiki/xacro" name="walrus_pod">
-	<xacro:macro name="walrus_pod" params="fb lr parent translateX translateY flipY robot_ns"> <!--fb : front, back ; lr: left, right -->
-		<link name="${robot_ns}/${fb}_${lr}_pod">
+	<xacro:macro name="walrus_pod" params="fb lr parent translateX translateY flipY tf_prefix"> <!--fb : front, back ; lr: left, right -->
+		<link name="${tf_prefix}${fb}_${lr}_pod">
 			<inertial>
 				<mass value="${pod_mass}" />
@@ -25,25 +25,25 @@
 			</collision>
 		</link>
-		<gazebo reference="${robot_ns}/${fb}_${lr}_pod">
+		<gazebo reference="${tf_prefix}${fb}_${lr}_pod">
 			<material>Gazebo/FlatBlack</material>
 			<turnGravityOff>false</turnGravityOff>
 		</gazebo>
-		<joint name="${robot_ns}/${fb}_${lr}_pod_joint" type="continuous">
+		<joint name="${tf_prefix}${fb}_${lr}_pod_joint" type="continuous">
 			<parent link="${parent}"/>
-			<child link="${robot_ns}/${fb}_${lr}_pod"/>
+			<child link="${tf_prefix}${fb}_${lr}_pod"/>
 			<origin xyz="${translateX * center_tread_inner_length/2} ${translateY * (base_y_size/2+tread_width/2+tread_width)} ${-base_z_to_pod_origin}" rpy="0 ${M_PI/2-M_PI/2*translateX} 0" />
 			<axis xyz="0 1 0" rpy="0 0 0" />
 			<joint_properties damping="0.0" friction="0.0"/>
 		</joint>
-		<transmission name="${robot_ns}/${fb}_${lr}_pod_joint_trans">
+		<transmission name="${tf_prefix}${fb}_${lr}_pod_joint_trans">
 			<type>transmission_interface/SimpleTransmission</type>
-			<joint name="${robot_ns}/${fb}_${lr}_pod_joint">
+			<joint name="${tf_prefix}${fb}_${lr}_pod_joint">
 				<hardwareInterface>hardware_interface/EffortJointInterface</hardwareInterface>
 			</joint>
-			<actuator name="${robot_ns}/${fb}_${lr}_pod_joint_actuator">
+			<actuator name="${tf_prefix}${fb}_${lr}_pod_joint_actuator">
 				<mechanicalReduction>1</mechanicalReduction>
 			</actuator>
 		</transmission>
-		<link name="${robot_ns}/${fb}_${lr}_pod_drive_cylinder">
+		<link name="${tf_prefix}${fb}_${lr}_pod_drive_cylinder">
 			<inertial>
 				<mass value="${tread_cylinder_mass}" />
@@ -74,12 +74,12 @@
 			</collision>
 		</link>
-		<joint name="${robot_ns}/${fb}_${lr}_pod_drive_joint" type="continuous">
-			<parent link="${robot_ns}/${fb}_${lr}_pod"/>
-			<child link="${robot_ns}/${fb}_${lr}_pod_drive_cylinder"/>
+		<joint name="${tf_prefix}${fb}_${lr}_pod_drive_joint" type="continuous">
+			<parent link="${tf_prefix}${fb}_${lr}_pod"/>
+			<child link="${tf_prefix}${fb}_${lr}_pod_drive_cylinder"/>
 			<origin xyz="0 0 0" rpy="${M_PI/2} 0 0" />
 			<axis xyz="0 0 1" rpy="0 0 0" />
-			<mimic joint="${robot_ns}/${lr}_drive_joint" multiplier="1.0" offset="0.0" />
+			<mimic joint="${tf_prefix}${lr}_drive_joint" multiplier="1.0" offset="0.0" />
 		</joint>
-		<link name="${robot_ns}/${fb}_${lr}_pod_drive_idler_cylinder">
+		<link name="${tf_prefix}${fb}_${lr}_pod_drive_idler_cylinder">
 			<inertial>
 				<mass value="${tread_cylinder_mass}" />
@@ -110,10 +110,10 @@
 			</collision>
 		</link>
-		<joint name="${robot_ns}/${fb}_${lr}_pod_drive_idler_joint" type="continuous">
-			<parent link="${robot_ns}/${fb}_${lr}_pod"/>
-			<child link="${robot_ns}/${fb}_${lr}_pod_drive_idler_cylinder"/>
+		<joint name="${tf_prefix}${fb}_${lr}_pod_drive_idler_joint" type="continuous">
+			<parent link="${tf_prefix}${fb}_${lr}_pod"/>
+			<child link="${tf_prefix}${fb}_${lr}_pod_drive_idler_cylinder"/>
 			<origin xyz="${pod_inner_length} 0 0" rpy="${M_PI/2} 0 0" />
 			<axis xyz="0 0 1" rpy="0 0 0" />
-			<mimic joint="${robot_ns}/${lr}_drive_joint" multiplier="1.0" offset="0.0" />
+			<mimic joint="${tf_prefix}${lr}_drive_joint" multiplier="1.0" offset="0.0" />
 		</joint>
   	</xacro:macro>

Commit message: Began adding boom to robot model Added kinect sensor

File: walrus_description/robots/walrus.urdf.xacro (robot description, xacro)
@@ -5,5 +5,5 @@
   <property name="tf_prefix" value="$(arg tf_prefix)" />
   <property name="robot_ns" value="$(arg robot_ns)" />
-  <xacro:walrus tf_prefix="${tf_prefix}"/>
+  <xacro:walrus tf_prefix="${tf_prefix}" robot_ns="${robot_ns}"/>
   <gazebo>
     <plugin name="gazebo_ros_control" filename="libgazebo_ros_control.so">

File: walrus_description/urdf/base.urdf.xacro (robot description, xacro)
@@ -62,5 +62,6 @@
     <xacro:include filename="$(find walrus_description)/urdf/pod.urdf.xacro" />
     <xacro:include filename="$(find walrus_description)/urdf/center_tread.urdf.xacro" />
-    <xacro:macro name="walrus" params="tf_prefix">
+    <xacro:include filename="$(find walrus_description)/urdf/boom.urdf.xacro" />
+    <xacro:macro name="walrus" params="tf_prefix robot_ns">
       <!-- BASE-FOOTPRINT -->
       <link name="${tf_prefix}base_footprint">
@@ -113,4 +114,5 @@
       <walrus_center_tread lr="left" parent="${tf_prefix}base_link" translateY="1" flipY="-1" tf_prefix="${tf_prefix}"/>
       <walrus_center_tread lr="right" parent="${tf_prefix}base_link" translateY="-1" flipY="-1" tf_prefix="${tf_prefix}"/>
+      <walrus_boom parent="${tf_prefix}base_link" tf_prefix="${tf_prefix}boom/" robot_ns="${robot_ns}/boom"/>
       <transmission name="${tf_prefix}left_drive_trans">
         <type>transmission_interface/SimpleTransmission</type>
