Commit message: Created drive controller (currently just a diff drive controller) Added last components of web interface backend to drive robot #19

File: walrus_description/urdf/center_tread.urdf.xacro (robot description, xacro)
@@ -61,5 +61,5 @@
 			<parent link="${tf_prefix}${lr}_center_tread"/>
 			<child link="${tf_prefix}${lr}_center_tread_front_cylinder"/>
-			<origin xyz="${center_tread_inner_length/2} 0 0" rpy="${M_PI/2} 0 0" />
+			<origin xyz="${center_tread_inner_length/2} 0 0" rpy="${-M_PI/2} 0 0" />
 			<axis xyz="0 0 1" rpy="0 0 0" />
 		</joint>
@@ -96,5 +96,5 @@
 			<parent link="${tf_prefix}${lr}_center_tread"/>
 			<child link="${tf_prefix}${lr}_center_tread_back_cylinder"/>
-			<origin xyz="${-center_tread_inner_length/2} 0 0" rpy="${M_PI/2} 0 0" />
+			<origin xyz="${-center_tread_inner_length/2} 0 0" rpy="${-M_PI/2} 0 0" />
 			<axis xyz="0 0 1" rpy="0 0 0" />
 			<mimic joint="${tf_prefix}${lr}_drive_joint" multiplier="1.0" offset="0.0" />

File: walrus_description/urdf/pod.urdf.xacro (robot description, xacro)
@@ -77,5 +77,5 @@
 			<parent link="${tf_prefix}${fb}_${lr}_pod"/>
 			<child link="${tf_prefix}${fb}_${lr}_pod_drive_cylinder"/>
-			<origin xyz="0 0 0" rpy="${M_PI/2} 0 0" />
+			<origin xyz="0 0 0" rpy="${-M_PI/2} 0 0" />
 			<axis xyz="0 0 1" rpy="0 0 0" />
 			<mimic joint="${tf_prefix}${lr}_drive_joint" multiplier="1.0" offset="0.0" />
@@ -113,5 +113,5 @@
 			<parent link="${tf_prefix}${fb}_${lr}_pod"/>
 			<child link="${tf_prefix}${fb}_${lr}_pod_drive_idler_cylinder"/>
-			<origin xyz="${pod_inner_length} 0 0" rpy="${M_PI/2} 0 0" />
+			<origin xyz="${pod_inner_length} 0 0" rpy="${-M_PI/2} 0 0" />
 			<axis xyz="0 0 1" rpy="0 0 0" />
 			<mimic joint="${tf_prefix}${lr}_drive_joint" multiplier="1.0" offset="0.0" />
