Commit message: Updated physical properties to behave better Removed extra transmissions in urdf and added mimic for fake joints

File: walrus_description/urdf/base.urdf.xacro (robot description, xacro)
@@ -49,14 +49,14 @@
     <property name="center_tread_iyz_com_cs" value="0"/>
     <property name="center_tread_izz_com_cs" value="1"/>
-    <property name="tread_cylinder_mass" value="0.5" />
+    <property name="tread_cylinder_mass" value="1"/>
     <property name="tread_cylinder_x_com" value="0"/>
     <property name="tread_cylinder_y_com" value="0"/>
     <property name="tread_cylinder_z_com" value="0"/>
-    <property name="tread_cylinder_ixx_com_cs" value="0.001"/>
+    <property name="tread_cylinder_ixx_com_cs" value="1"/>
     <property name="tread_cylinder_ixy_com_cs" value="0"/>
     <property name="tread_cylinder_ixz_com_cs" value="0"/>
-    <property name="tread_cylinder_iyy_com_cs" value="0.001"/>
+    <property name="tread_cylinder_iyy_com_cs" value="1"/>
     <property name="tread_cylinder_iyz_com_cs" value="0"/>
-    <property name="tread_cylinder_izz_com_cs" value="0.001"/>
+    <property name="tread_cylinder_izz_com_cs" value="1"/>
     <xacro:include filename="$(find walrus_description)/urdf/simple_transform.urdf.xacro" />
     <xacro:include filename="$(find walrus_description)/urdf/pod.urdf.xacro" />

File: walrus_description/urdf/center_tread.urdf.xacro (robot description, xacro)
@@ -58,5 +58,5 @@
 			</collision>
 		</link>
-		<joint name="${robot_ns}/${lr}_center_tread_front_cylinder_joint" type="continuous">
+		<joint name="${robot_ns}/${lr}_drive_joint" type="continuous">
 			<parent link="${robot_ns}/${lr}_center_tread"/>
 			<child link="${robot_ns}/${lr}_center_tread_front_cylinder"/>
@@ -98,21 +98,6 @@
 			<origin xyz="${-center_tread_inner_length/2} 0 0" rpy="${M_PI/2} 0 0" />
 			<axis xyz="0 0 1" rpy="0 0 0" />
+			<mimic joint="${robot_ns}/${lr}_drive_joint" multiplier="1.0" offset="0.0" />
 		</joint>
-		<transmission name="${robot_ns}/${lr}_center_tread_drive_back_trans">
-			<type>transmission_interface/SimpleTransmission</type>
-			<joint name="${robot_ns}/${lr}_center_tread_back_cylinder_joint"/>
-			<actuator name="${robot_ns}/${lr}_pod_drive_actuator">
-				<hardwareInterface>EffortJointInterface</hardwareInterface>
-				<mechanicalReduction>1</mechanicalReduction>
-			</actuator>
-		</transmission>
-		<transmission name="${robot_ns}/${lr}_center_tread_drive_front_trans">
-			<type>transmission_interface/SimpleTransmission</type>
-			<joint name="${robot_ns}/${lr}_center_tread_front_cylinder_joint"/>
-			<actuator name="${robot_ns}/${lr}_pod_drive_actuator">
-				<hardwareInterface>EffortJointInterface</hardwareInterface>
-				<mechanicalReduction>1</mechanicalReduction>
-			</actuator>
-		</transmission>
   	</xacro:macro>
 </robot>

File: walrus_description/urdf/pod.urdf.xacro (robot description, xacro)
@@ -79,4 +79,5 @@
 			<origin xyz="0 0 0" rpy="${M_PI/2} 0 0" />
 			<axis xyz="0 0 1" rpy="0 0 0" />
+			<mimic joint="${robot_ns}/${lr}_drive_joint" multiplier="1.0" offset="0.0" />
 		</joint>
 		<link name="${robot_ns}/${fb}_${lr}_pod_extended_cylinder">
@@ -114,21 +115,6 @@
 			<origin xyz="${pod_inner_length} 0 0" rpy="${M_PI/2} 0 0" />
 			<axis xyz="0 0 1" rpy="0 0 0" />
+			<mimic joint="${robot_ns}/${lr}_drive_joint" multiplier="1.0" offset="0.0" />
 		</joint>
-		<transmission name="${robot_ns}/${fb}_${lr}_pod_drive_extended_trans">
-			<type>transmission_interface/SimpleTransmission</type>
-			<joint name="${robot_ns}/${fb}_${lr}_pod_extended_cylinder_joint"/>
-			<actuator name="${robot_ns}/${lr}_pod_drive_actuator">
-				<hardwareInterface>EffortJointInterface</hardwareInterface>
-				<mechanicalReduction>1</mechanicalReduction>
-			</actuator>
-		</transmission>
-		<transmission name="${robot_ns}/${fb}_${lr}_pod_drive_joint_trans">
-			<type>transmission_interface/SimpleTransmission</type>
-			<joint name="${robot_ns}/${fb}_${lr}_pod_joint_cylinder_joint"/>
-			<actuator name="${robot_ns}/${lr}_pod_drive_actuator">
-				<hardwareInterface>EffortJointInterface</hardwareInterface>
-				<mechanicalReduction>1</mechanicalReduction>
-			</actuator>
-		</transmission>
   	</xacro:macro>
 </robot>

Commit message: Added torque limits on pods Added more advanced pod controls Made mass properties more realistic

File: walrus_description/urdf/base.urdf.xacro (robot description, xacro)
@@ -33,10 +33,10 @@
     <property name="pod_y_com" value="0"/>
     <property name="pod_z_com" value="0"/>
-    <property name="pod_ixx_com_cs" value="1"/>
+    <property name="pod_ixx_com_cs" value="0.001"/>
     <property name="pod_ixy_com_cs" value="0"/>
     <property name="pod_ixz_com_cs" value="0"/>
-    <property name="pod_iyy_com_cs" value="1"/>
+    <property name="pod_iyy_com_cs" value="0.001"/>
     <property name="pod_iyz_com_cs" value="0"/>
-    <property name="pod_izz_com_cs" value="1"/>
+    <property name="pod_izz_com_cs" value="0.001"/>
     <property name="center_tread_mass" value="1" />
     <property name="center_tread_x_com" value="0"/>
@@ -53,10 +53,10 @@
     <property name="tread_cylinder_y_com" value="0"/>
     <property name="tread_cylinder_z_com" value="0"/>
-    <property name="tread_cylinder_ixx_com_cs" value="1"/>
+    <property name="tread_cylinder_ixx_com_cs" value="0.01"/>
     <property name="tread_cylinder_ixy_com_cs" value="0"/>
     <property name="tread_cylinder_ixz_com_cs" value="0"/>
-    <property name="tread_cylinder_iyy_com_cs" value="1"/>
+    <property name="tread_cylinder_iyy_com_cs" value="0.01"/>
     <property name="tread_cylinder_iyz_com_cs" value="0"/>
-    <property name="tread_cylinder_izz_com_cs" value="1"/>
+    <property name="tread_cylinder_izz_com_cs" value="0.01"/>
     <xacro:include filename="$(find walrus_description)/urdf/simple_transform.urdf.xacro" />
     <xacro:include filename="$(find walrus_description)/urdf/pod.urdf.xacro" />

File: walrus_description/urdf/pod.urdf.xacro (robot description, xacro)
@@ -34,5 +34,4 @@
 			<origin xyz="${translateX * center_tread_inner_length/2} ${translateY * (base_y_size/2+tread_width/2+tread_width)} ${-base_z_to_pod_origin}" rpy="0 ${M_PI/2-M_PI/2*translateX} 0" />
 			<axis xyz="0 1 0" rpy="0 0 0" />
-			<limit effort="100" velocity="100"/>
 			<joint_properties damping="0.0" friction="0.0"/>
 		</joint>

Commit message: Added IMU to gazebo model

File: walrus_description/urdf/base.urdf.xacro (robot description, xacro)
@@ -108,4 +108,18 @@
 	<turnGravityOff>false</turnGravityOff>
       </gazebo>
+      <joint name="${tf_prefix}imu_joint" type="fixed">
+	<origin xyz="0 0 0" rpy="0 0 0" />
+	<parent link="${tf_prefix}base_link"/>
+	<child link="${tf_prefix}imu" />
+      </joint>
+      <link name="${tf_prefix}imu"/>
+      <gazebo>
+	  <plugin name="imu_controller" filename="libgazebo_ros_imu.so">
+	    <topicName>${robot_ns}/imu/data</topicName>
+	    <serviceName>${robot_ns}/data/calibrate</serviceName>
+	    <bodyName>${tf_prefix}imu</bodyName>
+	    <updateRate>50</updateRate>
+	  </plugin>
+      </gazebo>
       <walrus_pod fb="back" lr="left" parent="${tf_prefix}base_link" translateX="-1" translateY="1" flipY="-1" tf_prefix="${tf_prefix}"/>
       <walrus_pod fb="back" lr="right" parent="${tf_prefix}base_link" translateX="-1" translateY="-1" flipY="-1" tf_prefix="${tf_prefix}"/>

Commit message: Added cameras to robot model

File: walrus_description/urdf/base.urdf.xacro (robot description, xacro)
@@ -63,4 +63,5 @@
     <xacro:include filename="$(find walrus_description)/urdf/center_tread.urdf.xacro" />
     <xacro:include filename="$(find walrus_description)/urdf/boom.urdf.xacro" />
+    <xacro:include filename="$(find walrus_description)/urdf/simple_camera.urdf.xacro" />
     <xacro:macro name="walrus" params="tf_prefix robot_ns">
       <!-- BASE-FOOTPRINT -->
@@ -129,4 +130,10 @@
       <walrus_center_tread lr="right" parent="${tf_prefix}base_link" translateY="-1" flipY="-1" tf_prefix="${tf_prefix}"/>
       <walrus_boom parent="${tf_prefix}base_link" tf_prefix="${tf_prefix}boom/" robot_ns="${robot_ns}/boom"/>
+      <simple_camera parent="${tf_prefix}base_link" tf_prefix="${tf_prefix}front_camera" camera_ns="${robot_ns}/front_camera" name="front_camera">
+	<origin xyz="0.08 0 0" rpy="0 0 0" />
+      </simple_camera>
+      <simple_camera parent="${tf_prefix}base_link" tf_prefix="${tf_prefix}back_camera" camera_ns="${robot_ns}/back_camera" name="back_camera">
+	<origin xyz="-0.08 0 0" rpy="0 0 ${M_PI}" />
+      </simple_camera>
       <transmission name="${tf_prefix}left_drive_trans">
         <type>transmission_interface/SimpleTransmission</type>

Commit message: Did some robot description cleanup

File: walrus_description/urdf/base.urdf.xacro (robot description, xacro)
@@ -123,11 +123,13 @@
 	  </plugin>
       </gazebo>
+      <!-- Center Treads -->
+      <walrus_center_tread lr="left" parent="${tf_prefix}base_link" translateY="1" flipY="-1" tf_prefix="${tf_prefix}"/>
+      <walrus_center_tread lr="right" parent="${tf_prefix}base_link" translateY="-1" flipY="-1" tf_prefix="${tf_prefix}"/>
+      <!-- Pods -->
       <walrus_pod fb="back" lr="left" parent="${tf_prefix}base_link" translateX="-1" translateY="1" flipY="-1" tf_prefix="${tf_prefix}"/>
       <walrus_pod fb="back" lr="right" parent="${tf_prefix}base_link" translateX="-1" translateY="-1" flipY="-1" tf_prefix="${tf_prefix}"/>
       <walrus_pod fb="front" lr="left" parent="${tf_prefix}base_link" translateX="1" translateY="1" flipY="-1" tf_prefix="${tf_prefix}"/>
       <walrus_pod fb="front" lr="right" parent="${tf_prefix}base_link" translateX="1" translateY="-1" flipY="-1" tf_prefix="${tf_prefix}"/>
-      <walrus_center_tread lr="left" parent="${tf_prefix}base_link" translateY="1" flipY="-1" tf_prefix="${tf_prefix}"/>
-      <walrus_center_tread lr="right" parent="${tf_prefix}base_link" translateY="-1" flipY="-1" tf_prefix="${tf_prefix}"/>
-      <walrus_boom parent="${tf_prefix}base_link" tf_prefix="${tf_prefix}boom/" robot_ns="${robot_ns}/boom"/>
+      <!-- Cameras -->
       <simple_camera parent="${tf_prefix}base_link" tf_prefix="${tf_prefix}front_camera" camera_ns="${robot_ns}/front_camera" name="front_camera">
 	<origin xyz="0.08 0 0" rpy="0 0 0" />
@@ -136,22 +138,6 @@
 	<origin xyz="-0.08 0 0" rpy="0 0 ${M_PI}" />
       </simple_camera>
-      <transmission name="${tf_prefix}left_drive_trans">
-        <type>transmission_interface/SimpleTransmission</type>
-        <joint name="${tf_prefix}left_drive_joint">
-          <hardwareInterface>hardware_interface/EffortJointInterface</hardwareInterface>
-	</joint>
-        <actuator name="${tf_prefix}left_drive_actuator">
-          <mechanicalReduction>1</mechanicalReduction>
-        </actuator>
-      </transmission>
-      <transmission name="${tf_prefix}right_drive_trans">
-        <type>transmission_interface/SimpleTransmission</type>
-        <joint name="${tf_prefix}right_drive_joint">
-          <hardwareInterface>hardware_interface/EffortJointInterface</hardwareInterface>
-	</joint>
-        <actuator name="${tf_prefix}right_drive_actuator">
-          <mechanicalReduction>1</mechanicalReduction>
-        </actuator>
-      </transmission>
+      <!-- Boom -->
+      <walrus_boom parent="${tf_prefix}base_link" tf_prefix="${tf_prefix}boom/" robot_ns="${robot_ns}/boom"/>
     </xacro:macro>
 </robot>

File: walrus_description/urdf/boom.urdf.xacro (robot description, xacro)
@@ -3,4 +3,6 @@
         <xacro:include filename="$(find walrus_description)/urdf/kinectv2.urdf.xacro" />
 	<xacro:macro name="walrus_boom" params="parent tf_prefix robot_ns">
+		<!-- Boom base -->
+		<!-- Fixed base attached to the robot -->
 		<link name="${tf_prefix}base">
 			<inertial>
@@ -30,4 +32,6 @@
 			<origin xyz="-0.04 0 0.03" rpy="0 0 0" />
 		</joint>
+		<!-- Deploy base -->
+		<!-- Link that the deploy joint actuates (contains the pan actuator) -->
 		<link name="${tf_prefix}deploy_base">
 			<inertial>
@@ -59,4 +63,5 @@
 			<limit lower="${-M_PI/2}" upper="${M_PI/2}" effort="2" velocity="0.5" />
 		</joint>
+		<!-- Boom Mast -->
 		<link name="${tf_prefix}mast">
 			<inertial>
@@ -89,4 +94,6 @@
 			<limit lower="-2" upper="2" effort="2" velocity="0.5" />
 		</joint>
+		<!-- Tilt Base -->
+		<!-- Link actuated by the tilt motor -->
 		<link name="${tf_prefix}tilt_base">
 			<inertial>
@@ -118,4 +125,5 @@
 			<limit lower="${-M_PI/2}" upper="${M_PI/2}" effort="2" velocity="0.5" />
 		</joint>
+		<!-- Kinect -->
 		<kinectv2 parent="${tf_prefix}tilt_base" tf_prefix="${tf_prefix}kinect" camera_ns="${robot_ns}/kinect" name="boom_kinect">
 			<origin xyz="0 0 0.03" rpy="0 0 0" />

File: walrus_description/urdf/center_tread.urdf.xacro (robot description, xacro)
@@ -100,4 +100,13 @@
 			<mimic joint="${tf_prefix}${lr}_drive_joint" multiplier="1.0" offset="0.0" />
 		</joint>
+		<transmission name="${tf_prefix}${lr}_drive_trans">
+		  <type>transmission_interface/SimpleTransmission</type>
+		  <joint name="${tf_prefix}${lr}_drive_joint">
+		    <hardwareInterface>hardware_interface/EffortJointInterface</hardwareInterface>
+		  </joint>
+		  <actuator name="${tf_prefix}${lr}_drive_actuator">
+		    <mechanicalReduction>1</mechanicalReduction>
+		  </actuator>
+		</transmission>
   	</xacro:macro>
 </robot>

Commit message: Updated lots of robot measurements

File: walrus_description/urdf/base.urdf.xacro (robot description, xacro)
@@ -16,13 +16,16 @@
     <property name="base_iyz_com_cs" value="0"/>
     <property name="base_izz_com_cs" value="1"/>
-    <property name="base_x_size" value="0.1375"/>
-    <property name="base_y_size" value="0.13"/>
-    <property name="base_z_size" value="0.031"/>
-    <property name="tread_radius" value="0.044"/>
-    <property name="tread_width" value="0.0381"/>
-    <property name="pod_inner_length" value="0.1041"/>
-    <property name="center_tread_inner_length" value="0.2794"/>
-    <property name="base_z_to_pod_origin" value="0.006" />
-    <property name="tread_body_inset" value="0.03" />
+    <property name="base_x_size" value="0.635"/>
+    <property name="base_y_size" value="0.2667"/>
+    <property name="base_z_size" value="0.181"/>
+    <property name="tread_radius" value="0.0765"/>
+    <property name="tread_pod_idler_radius" value="0.039875"/>
+    <property name="tread_width" value="0.05"/>
+    <property name="pod_inner_length" value="0.2647"/>
+    <property name="center_tread_inner_length" value="0.4826"/>
+    <property name="center_tread_body_offset" value="0.00199"/>
+    <property name="center_tread_pod_tread_offset" value="0.00159"/>
+    <property name="base_z_to_pod_origin" value="0.1302" />
+    <property name="tread_body_collision_inset" value="0.06" />
     <property name="tread_cylinder_mu1" value="1.0" />
     <property name="tread_cylinder_mu2" value="1.0" />
@@ -92,5 +95,5 @@
 	</inertial>
 	<visual>
-	  <origin xyz="0 0 0" rpy="0 0 0" />
+	  <origin xyz="0 0 ${-base_z_size/2}" rpy="0 0 0" />
 	  <geometry>
 	    <box size = "${base_x_size} ${base_y_size} ${base_z_size}"/>
@@ -99,5 +102,5 @@
 	</visual>
 	<collision>
-	  <origin xyz="0 0 0" rpy="0 0 0" />
+	  <origin xyz="0 0 ${-base_z_size/2}" rpy="0 0 0" />
 	  <geometry>
 	    <box size = "${base_x_size} ${base_y_size} ${base_z_size}"/>
@@ -133,8 +136,11 @@
       <!-- Cameras -->
       <simple_camera parent="${tf_prefix}base_link" tf_prefix="${tf_prefix}front_camera" camera_ns="${robot_ns}/front_camera" name="front_camera">
-	<origin xyz="0.08 0 0" rpy="0 0 0" />
+	<origin xyz="0.307 0.0185 -0.0519" rpy="0 0 0" />
       </simple_camera>
       <simple_camera parent="${tf_prefix}base_link" tf_prefix="${tf_prefix}back_camera" camera_ns="${robot_ns}/back_camera" name="back_camera">
-	<origin xyz="-0.08 0 0" rpy="0 0 ${M_PI}" />
+	<origin xyz="-0.307 -0.0185 -0.0519" rpy="0 0 ${M_PI}" />
+      </simple_camera>
+      <simple_camera parent="${tf_prefix}base_link" tf_prefix="${tf_prefix}bottom_camera" camera_ns="${robot_ns}/bottom_camera" name="bottom_camera">
+	<origin xyz="-0.196 0.01197 -0.166" rpy="0 0.49 0" />
       </simple_camera>
       <!-- Boom -->

File: walrus_description/urdf/boom.urdf.xacro (robot description, xacro)
@@ -30,5 +30,5 @@
 			<parent link="${parent}"/>
 			<child link="${tf_prefix}base"/>
-			<origin xyz="-0.04 0 0.03" rpy="0 0 0" />
+			<origin xyz="-0.23 0 0.03" rpy="0 0 0" />
 		</joint>
 		<!-- Deploy base -->

File: walrus_description/urdf/center_tread.urdf.xacro (robot description, xacro)
@@ -20,5 +20,5 @@
 			<collision>
 				<geometry>
-			                <box size = "${center_tread_inner_length} ${tread_width} ${(tread_radius-tread_body_inset)*2}"/>
+			                <box size = "${center_tread_inner_length} ${tread_width} ${(tread_radius-tread_body_collision_inset)*2}"/>
 				</geometry>
 			</collision>
@@ -27,5 +27,5 @@
 			<parent link="${parent}"/>
 			<child link="${tf_prefix}${lr}_center_tread"/>
-			<origin xyz="0 ${translateY * (base_y_size/2+tread_width/2)} ${-base_z_to_pod_origin}" rpy="0 0 0" />
+			<origin xyz="0 ${translateY * (base_y_size/2+tread_width/2+center_tread_body_offset)} ${-base_z_to_pod_origin}" rpy="0 0 0" />
 		</joint>
 		<link name="${tf_prefix}${lr}_center_tread_front_cylinder">
@@ -106,5 +106,5 @@
 		  </joint>
 		  <actuator name="${tf_prefix}${lr}_drive_actuator">
-		    <mechanicalReduction>${flipY * 12 * 2.5 * 60}</mechanicalReduction><!-- gearbox: 12, chain: 2.5, is in rpm: 60 -->
+		    <mechanicalReduction>${flipY * 12 * 2.5 * 60 / (M_PI * 2)}</mechanicalReduction><!-- gearbox: 12, chain: 2.5, is in rpm: 60 / 2pi,  -->
 		  </actuator>
 		</transmission>

File: walrus_description/urdf/pod.urdf.xacro (robot description, xacro)
@@ -12,5 +12,5 @@
 				<origin xyz="${pod_inner_length/2} 0 0" rpy="${flipY*M_PI} 0 0" />
 				<geometry>
-			                <box size = "${pod_inner_length} ${tread_width} ${tread_radius*2}"/>
+			                <box size = "${pod_inner_length} ${tread_width} ${tread_pod_idler_radius*2}"/>
 				</geometry>
 				<material name="blue">
@@ -21,5 +21,5 @@
 				<origin xyz="${pod_inner_length/2} 0 0" rpy="${flipY*M_PI} 0 0" />
 				<geometry>
-			                <box size = "${pod_inner_length} ${tread_width} ${(tread_radius-tread_body_inset)*2}"/>
+			                <box size = "${pod_inner_length} ${tread_width} ${(tread_radius-tread_body_collision_inset)*2}"/>
 				</geometry>
 			</collision>
@@ -32,5 +32,5 @@
 			<parent link="${parent}"/>
 			<child link="${tf_prefix}${fb}_${lr}_pod"/>
-			<origin xyz="${translateX * center_tread_inner_length/2} ${translateY * (base_y_size/2+tread_width/2+tread_width)} ${-base_z_to_pod_origin}" rpy="0 ${M_PI/2-M_PI/2*translateX} 0" />
+			<origin xyz="${translateX * center_tread_inner_length/2} ${translateY * (base_y_size/2+tread_width/2+center_tread_body_offset+tread_width+center_tread_pod_tread_offset)} ${-base_z_to_pod_origin}" rpy="0 ${M_PI/2-M_PI/2*translateX} 0" />
 			<axis xyz="0 1 0" rpy="0 0 0" />
 			<joint_properties damping="0.0" friction="0.0"/>
@@ -90,5 +90,5 @@
 			<visual>
 				<geometry>
-					<cylinder length="${tread_width}" radius="${tread_radius}" />
+					<cylinder length="${tread_width}" radius="${tread_pod_idler_radius}" />
 				</geometry>
 				<material name="red">
@@ -98,5 +98,5 @@
 			<collision>
 				<geometry>
-					<cylinder length="${tread_width}" radius="${tread_radius}" />
+					<cylinder length="${tread_width}" radius="${tread_pod_idler_radius}" />
 				</geometry>
 				<friction>

File: walrus_description/urdf/simple_camera.urdf.xacro (robot description, xacro)
@@ -10,5 +10,5 @@
 			</inertial>
 			<visual>
-				<origin xyz="0 0 0" rpy="0 ${M_PI/2} 0" />
+				<origin xyz="-0.025 0 0" rpy="0 ${M_PI/2} 0" />
 				<geometry>
 			                <cylinder length="0.05" radius="0.01"/>
@@ -19,5 +19,5 @@
 			</visual>
 			<collision>
-				<origin xyz="0 0 0" rpy="0 ${M_PI/2} 0" />
+				<origin xyz="-0.025 0 0" rpy="0 ${M_PI/2} 0" />
 				<geometry>
 			                <cylinder length="0.05" radius="0.01"/>
