Commit message: Added robot meshes

File: walrus_description/urdf/base.urdf.xacro (robot description, xacro)
@@ -95,9 +95,11 @@
 	</inertial>
 	<visual>
-	  <origin xyz="0 0 ${-base_z_size/2}" rpy="0 0 0" />
-	  <geometry>
-	    <box size = "${base_x_size} ${base_y_size} ${base_z_size}"/>
-	  </geometry>
-	  <material name="Black" />
+	  <origin xyz="0 0 0" rpy="0 0 0" />
+          <geometry>
+            <mesh filename="package://walrus_description/meshes/base.stl" />
+          </geometry>
+	  <material name="Red">
+	    <color rgba=".4 0 0 1"/>
+	  </material>
 	</visual>
 	<collision>
@@ -109,5 +111,5 @@
       </link>
       <gazebo reference="${tf_prefix}base_link">
-	<material>Gazebo/Green</material>
+	<material>Gazebo/Red</material>
 	<turnGravityOff>false</turnGravityOff>
       </gazebo>
@@ -130,7 +132,7 @@
       <walrus_center_tread lr="right" parent="${tf_prefix}base_link" translateY="-1" flipY="-1" tf_prefix="${tf_prefix}"/>
       <!-- Pods -->
-      <walrus_pod fb="back" lr="left" parent="${tf_prefix}base_link" translateX="-1" translateY="1" flipY="-1" tf_prefix="${tf_prefix}"/>
+      <walrus_pod fb="back" lr="left" parent="${tf_prefix}base_link" translateX="-1" translateY="1" flipY="1" tf_prefix="${tf_prefix}"/>
       <walrus_pod fb="back" lr="right" parent="${tf_prefix}base_link" translateX="-1" translateY="-1" flipY="-1" tf_prefix="${tf_prefix}"/>
-      <walrus_pod fb="front" lr="left" parent="${tf_prefix}base_link" translateX="1" translateY="1" flipY="-1" tf_prefix="${tf_prefix}"/>
+      <walrus_pod fb="front" lr="left" parent="${tf_prefix}base_link" translateX="1" translateY="1" flipY="1" tf_prefix="${tf_prefix}"/>
       <walrus_pod fb="front" lr="right" parent="${tf_prefix}base_link" translateX="1" translateY="-1" flipY="-1" tf_prefix="${tf_prefix}"/>
       <!-- Cameras -->

File: walrus_description/urdf/center_tread.urdf.xacro (robot description, xacro)
@@ -10,10 +10,10 @@
 			</inertial>
 			<visual>
-				<origin xyz="0 0 0" rpy="${flipY*M_PI} 0 0" />
+				<origin xyz="0 0 0" rpy="0 0 0" />
 				<geometry>
-			                <box size = "${center_tread_inner_length} ${tread_width} ${tread_radius*2}"/>
+				  <mesh filename="package://walrus_description/meshes/${lr}_center_tread.stl"/>
 				</geometry>
-				<material name="blue">
-					<color rgba="0 0 0.8 1"/>
+				<material name="Grey">
+				  <color rgba=".2 .2 .2 1"/>
 				</material>
 			</visual>
@@ -24,4 +24,8 @@
 			</collision>
 		</link>
+		<gazebo reference="${tf_prefix}${lr}_center_tread">
+			<material>Gazebo/DarkGrey</material>
+			<turnGravityOff>false</turnGravityOff>
+		</gazebo>
 		<joint name="${tf_prefix}${lr}_center_tread_joint" type="fixed">
 			<parent link="${parent}"/>
@@ -36,12 +40,4 @@
 					 iyy="${tread_cylinder_iyy_com_cs}" iyz="${tread_cylinder_iyz_com_cs}" izz="${tread_cylinder_izz_com_cs}" />
 			</inertial>
-		<visual>
-				<geometry>
-					<cylinder length="${tread_width}" radius="${tread_radius}" />
-				</geometry>
-				<material name="red">
-					<color rgba="0.8 0 0 1"/>
-				</material>
-			</visual>
 			<collision>
 				<geometry>
@@ -71,12 +67,4 @@
 					 iyy="${tread_cylinder_iyy_com_cs}" iyz="${tread_cylinder_iyz_com_cs}" izz="${tread_cylinder_izz_com_cs}" />
 			</inertial>
-			<visual>
-				<geometry>
-					<cylinder length="${tread_width}" radius="${tread_radius}" />
-				</geometry>
-				<material name="red">
-					<color rgba="0.8 0 0 1"/>
-				</material>
-			</visual>
 			<collision>
 				<geometry>

File: walrus_description/urdf/pod.urdf.xacro (robot description, xacro)
@@ -10,10 +10,10 @@
 			</inertial>
 			<visual>
-				<origin xyz="${pod_inner_length/2} 0 0" rpy="${flipY*M_PI} 0 0" />
+				<origin xyz="0 0 0" rpy="${M_PI/2 - flipY*M_PI/2} 0 0" />
 				<geometry>
-			                <box size = "${pod_inner_length} ${tread_width} ${tread_pod_idler_radius*2}"/>
+				  <mesh filename="package://walrus_description/meshes/pod.stl" />
 				</geometry>
-				<material name="blue">
-					<color rgba="0 0 0.8 1"/>
+				<material name="Red">
+				  <color rgba=".4 0 0 1"/>
 				</material>
 			</visual>
@@ -26,5 +26,5 @@
 		</link>
 		<gazebo reference="${tf_prefix}${fb}_${lr}_pod">
-			<material>Gazebo/FlatBlack</material>
+			<material>Gazebo/Red</material>
 			<turnGravityOff>false</turnGravityOff>
 		</gazebo>
@@ -52,12 +52,4 @@
 					 iyy="${tread_cylinder_iyy_com_cs}" iyz="${tread_cylinder_iyz_com_cs}" izz="${tread_cylinder_izz_com_cs}" />
 			</inertial>
-			<visual>
-				<geometry>
-					<cylinder length="${tread_width}" radius="${tread_radius}" />
-				</geometry>
-				<material name="red">
-					<color rgba="0.8 0 0 1"/>
-				</material>
-			</visual>
 			<collision>
 				<geometry>
@@ -88,12 +80,4 @@
 					 iyy="${tread_cylinder_iyy_com_cs}" iyz="${tread_cylinder_iyz_com_cs}" izz="${tread_cylinder_izz_com_cs}" />
 			</inertial>
-			<visual>
-				<geometry>
-					<cylinder length="${tread_width}" radius="${tread_pod_idler_radius}" />
-				</geometry>
-				<material name="red">
-					<color rgba="0.8 0 0 1"/>
-				</material>
-			</visual>
 			<collision>
 				<geometry>

Commit message: Made orientation display functional

File: walrus_description/urdf/base.urdf.xacro (robot description, xacro)
@@ -114,5 +114,5 @@
       </gazebo>
       <joint name="${tf_prefix}imu_joint" type="fixed">
-	<origin xyz="0 0 0" rpy="0 0 0" />
+	<origin xyz="0 0 0" rpy="${M_PI} 0 0" />
 	<parent link="${tf_prefix}base_link"/>
 	<child link="${tf_prefix}imu" />
@@ -120,5 +120,5 @@
       <link name="${tf_prefix}imu"/>
       <gazebo>
-	  <plugin name="imu_controller" filename="libgazebo_ros_imu.so">
+	  <plugin name="imu_controller" filename="libhector_gazebo_ros_imu.so">
 	    <topicName>${robot_ns}/imu/data</topicName>
 	    <serviceName>${robot_ns}/data/calibrate</serviceName>
